File: KiCad/RaspberryPi-SMI16.kicad_pcb (KiCad board)
At the start: 2 copper layers, 86 x 133.5 mm, 20 parts, among them J1 Screw_Terminal_01x02, U1 RASPBERRYPI_GPIO_40, U2 RFID-RC522

Commit message: change KiCad7
Other:
- net class Default removed

Commit message: SMI HAT PCB create
Parts:
- removed the REF** at (156.0, 159.0)
- added C3: C, Capacitor_SMD:C_0603_1608Metric, F.Cu at (178.0, 98.2)
- added J2: Conn_02x04_Odd_Even, MountingHole:MountingHole_3.2mm_M3, F.Cu at (229.5, 104.2)
- added J3: Screw_Terminal_01x18, Connector_PinHeader_2.54mm:PinHeader_1x18_P2.54mm_Vertical, F.Cu at (159.1, 114.5)
- added J4: Screw_Terminal_01x01, Connector_PinHeader_2.54mm:PinHeader_1x01_P2.54mm_Vertical, F.Cu at (215.0, 146.0)
- added R1: 330, Resistor_SMD:R_0603_1608Metric, F.Cu at (159.3, 107.8)
- added R10: 330, Resistor_SMD:R_0603_1608Metric, F.Cu at (181.9, 107.8)
- added R11: 330, Resistor_SMD:R_0603_1608Metric, F.Cu at (184.4, 107.8)
- added R12: 330, Resistor_SMD:R_0603_1608Metric, F.Cu at (186.8, 107.8)
- added R13: 330, Resistor_SMD:R_0603_1608Metric, F.Cu at (189.6, 107.8)
- added R14: 330, Resistor_SMD:R_0603_1608Metric, F.Cu at (192.0, 107.8)
- added R15: 330, Resistor_SMD:R_0603_1608Metric, F.Cu at (194.5, 107.8)
- added R16: 330, Resistor_SMD:R_0603_1608Metric, F.Cu at (197.0, 107.8)
- added R17: 330, Resistor_SMD:R_0603_1608Metric, F.Cu at (199.5, 107.8)
- added R18: 330, Resistor_SMD:R_0603_1608Metric, F.Cu at (202.0, 107.8)
- added R19: 330, Resistor_SMD:R_0603_1608Metric, F.Cu at (205.0, 107.2)
- added R2: 330, Resistor_SMD:R_0603_1608Metric, F.Cu at (161.8, 107.8)
- added R3: 330, Resistor_SMD:R_0603_1608Metric, F.Cu at (164.3, 107.8)
- added R4: 330, Resistor_SMD:R_0603_1608Metric, F.Cu at (166.8, 107.8)
- added R5: 330, Resistor_SMD:R_0603_1608Metric, F.Cu at (169.3, 107.8)
- added R6: 330, Resistor_SMD:R_0603_1608Metric, F.Cu at (171.8, 107.8)
- added R7: 330, Resistor_SMD:R_0603_1608Metric, F.Cu at (174.3, 107.8)
- added R8: 330, Resistor_SMD:R_0603_1608Metric, F.Cu at (176.8, 107.8)
- added R9: 330, Resistor_SMD:R_0603_1608Metric, F.Cu at (179.5, 107.8)
- added REF**: MountingHole_3.2mm_M3, MountingHole:MountingHole_3.2mm_M3, F.Cu at (160.5, 155.0)
- added REF**: MountingHole_3.2mm_M3, MountingHole:MountingHole_3.2mm_M3, F.Cu at (204.5, 155.0)
- added U3: 74HCT541, Package_SO:SOIC-20W_7.5x15.4mm_P1.27mm, F.Cu at (188.2, 97.9)
- C2: value CP -> C; footprint Capacitor_THT:CP_Radial_D8.0mm_P3.50mm -> Capacitor_SMD:C_0603_1608Metric; moved to F.Cu
- J1: footprint TerminalBlock:TerminalBlock_bornier-2_P5.08mm -> TerminalBlock_Phoenix:TerminalBlock_Phoenix_MKDS-1,5-2_1x02_P5.00mm_Horizontal
- JP1, JP2, RV1: moved to B.Cu
- R20: renamed from R1; moved to B.Cu
- U2: value RFID-RC522 -> 74HCT541; footprint library:RFID-RC522 -> Package_SO:SOIC-20W_7.5x12.8mm_P1.27mm; moved to F.Cu
- moved J1 70.3 mm to (146.0, 137.0), turned to 90 degrees
- moved C2 57.2 mm to (197.5, 98.3), turned to 90 degrees
- moved JP1 49.7 mm to (220.3, 69.0), turned to 0 degrees
- moved U2 49.2 mm to (170.0, 98.0)
- moved R20 44.2 mm to (220.0, 78.0), turned to -90 degrees
- moved JP2 41.6 mm to (220.3, 74.0), turned to 0 degrees
- moved C1 21.5 mm to (142.0, 112.0)
- moved RV1 5.25 mm to (212.0, 53.5), turned to 180 degrees
Connections:
- net Net-(DS1-Pad14) renamed LCD_D7
- net Net-(DS1-Pad4) renamed LCD_RS
- net Net-(U1-Pad31) renamed SOE
- BZ1 pad 1: Net-(BZ1-Pad1) -> Net-(BZ1--)
- C1 pad 1: +3V3 -> +5V
- DS1 pad 10: Net-(DS1-Pad10) -> unconnected-(DS1-D3-Pad10)
- DS1 pad 11: Net-(DS1-Pad11) -> LCD_D4
- DS1 pad 12: Net-(DS1-Pad12) -> LCD_D5
- DS1 pad 13: Net-(DS1-Pad13) -> LCD_D6
- DS1 pad 6: Net-(DS1-Pad6) -> LCD_E
- DS1 pad 7: Net-(DS1-Pad7) -> unconnected-(DS1-D0-Pad7)
- DS1 pad 8: Net-(DS1-Pad8) -> unconnected-(DS1-D1-Pad8)
- DS1 pad 9: Net-(DS1-Pad9) -> unconnected-(DS1-D2-Pad9)
- U1 pad 10: Net-(U1-Pad10) -> SD7
- U1 pad 11: Net-(U1-Pad11) -> SD9
- U1 pad 12: Net-(BZ1-Pad1) -> SD10
- U1 pad 15: Net-(DS1-Pad13) -> SD14
- U1 pad 16: Net-(U1-Pad16) -> SD15
- U1 pad 18: Net-(U1-Pad18) -> SD16
- U1 pad 19: Net-(U1-Pad19) -> SD2
- U1 pad 21: Net-(U1-Pad21) -> SD1
- U1 pad 22: Net-(U1-Pad22) -> SD17
- U1 pad 23: Net-(U1-Pad23) -> SD3
- U1 pad 24: Net-(U1-Pad24) -> SD0
- U1 pad 26: Net-(U1-Pad26) -> SWE
- U1 pad 27: Net-(U1-Pad27) -> unconnected-(U1-ID_SD-Pad27)
- U1 pad 28: Net-(U1-Pad28) -> unconnected-(U1-ID_SC-Pad28)
- U1 pad 29: Net-(U1-Pad29) -> LCD_E
- U1 pad 3: Net-(U1-Pad3) -> LCD_D4
- U1 pad 32: Net-(U1-Pad32) -> SD4
- U1 pad 33: Net-(U1-Pad33) -> SD5
- U1 pad 35: Net-(DS1-Pad6) -> SD11
- U1 pad 36: Net-(U1-Pad36) -> SD8
- U1 pad 38: Net-(DS1-Pad11) -> SD12
- U1 pad 40: Net-(DS1-Pad12) -> SD13
- U1 pad 5: Net-(U1-Pad5) -> LCD_D5
- U1 pad 7: Net-(U1-Pad7) -> LCD_D6
- U1 pad 8: Net-(U1-Pad8) -> SD6
- U2 pad 1: +3V3 -> GND
- U2 pad 2: Net-(U1-Pad22) -> SD7
- U2 pad 3: GND -> SD6
- U2 pad 4: Net-(U1-Pad18) -> SD5
- U2 pad 5: Net-(U1-Pad21) -> SD4
- U2 pad 6: Net-(U1-Pad19) -> SD3
- U2 pad 7: Net-(U1-Pad23) -> SD2
- U2 pad 8: Net-(U1-Pad24) -> SD1
Routing:
- net GND: track 310.2 -> 198.0 mm, vias 0 -> 2
- net SWE: track 0.00 -> 85.2 mm, vias 0 -> 1
- net Net-(U1-Pad24): track 79.8 -> 0.00 mm, vias 1 -> 0
- net SD16: track 0.00 -> 76.9 mm, vias 0 -> 1
- net SD13: track 0.00 -> 74.0 mm, vias 0 -> 1
- net Net-(U1-Pad23): track 72.9 -> 0.00 mm, vias 1 -> 0
- net SD17: track 0.00 -> 70.9 mm, vias 0 -> 1
- net LCD_D5: track 0.00 -> 70.4 mm, vias 0 -> 2
- net LCD_D4: track 0.00 -> 69.6 mm, vias 0 -> 2
- net LCD_D6: track 0.00 -> 69.6 mm, vias 0 -> 2
- net SD10: track 0.00 -> 67.7 mm, vias 0 -> 3
- net Net-(U1-Pad19): track 64.8 -> 0.00 mm, vias 1 -> 0
- net Net-(BZ1-Pad1): track 63.8 -> 0.00 mm
- net Net-(U1-Pad21): track 63.6 -> 0.00 mm, vias 1 -> 0
- net SD12: track 0.00 -> 63.4 mm, vias 0 -> 1
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- added copper zone on B.Cu, net GND
- added copper zone on F.Cu, net GND
Other:
- board text added: "GND 5V"
